File: eth-uart.sch (EAGLE design)
At the start: 40 parts, among them IC1 STM32F407VE, IC2 DP83848, IC3 LDS3985M33R, X5 USBMICRO_B, X7 B78477P1001A314

Commit message: boot0 on solidjump
Parts:
- added SJ1: (no value), netcat:SJ3
Connections:
- net N$1 renamed LED_G
- net N$10 renamed LED_Y
- net N$42 renamed LED_LINK
- net N$43 renamed LED_ACT
- new net BOOT0: IC1SPEC.BOOT0, SJ1.2
- net 3.3V: now also SJ1.3
- net GND: now also SJ1.1; no longer IC1SPEC.BOOT0
Changed lines of the file:
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@@
 <part name="R10" library="netcat" deviceset="RES" device="R0402" value="4.7k"/>
 <part name="GND15" library="netcat" deviceset="GND" device=""/>
+<part name="SJ1" library="netcat" deviceset="SJ3" device=""/>
 </parts>
 <sheets>
@@
 <instance part="C8" gate="G$1" x="-71.12" y="-160.02"/>
 <instance part="C9" gate="G$1" x="-78.74" y="-160.02"/>
-<instance part="3.3V1" gate="G$1" x="-71.12" y="-101.6" smashed="yes" rot="R180">
-<attribute name="VALUE" x="-76.2" y="-101.6" size="1.778" layer="96" rot="R180"/>
+<instance part="3.3V1" gate="G$1" x="-86.36" y="-96.52" smashed="yes" rot="R180">
+<attribute name="VALUE" x="-91.44" y="-96.52" size="1.778" layer="96" rot="R180"/>
 </instance>
 <instance part="3.3V2" gate="G$1" x="-76.2" y="-132.08" smashed="yes" rot="R180">
@@
 <instance part="GND6" gate="GND" x="-83.82" y="-149.86"/>
 <instance part="GND7" gate="GND" x="33.02" y="-177.8"/>
-<instance part="GND8" gate="GND" x="-71.12" y="-111.76"/>
+<instance part="GND8" gate="GND" x="-83.82" y="-114.3"/>
 <instance part="OSC1" gate="G$1" x="78.74" y="-165.1"/>
 <instance part="GND9" gate="GND" x="71.12" y="-172.72"/>
@@
 <instance part="R10" gate="G$1" x="147.32" y="-144.78"/>
 <instance part="GND15" gate="GND" x="154.94" y="-149.86"/>
+<instance part="SJ1" gate="G$1" x="-76.2" y="-104.14" rot="R180"/>
 </instances>
 <busses>
@@
 </segment>
 <segment>
-<wire x1="-68.58" y1="-104.14" x2="-71.12" y2="-104.14" width="0.1524" layer="91"/>
-<wire x1="-71.12" y1="-104.14" x2="-71.12" y2="-109.22" width="0.1524" layer="91"/>
-<pinref part="IC1" gate="SPEC" pin="BOOT0"/>
 <pinref part="GND8" gate="GND" pin="GND"/>
+<pinref part="SJ1" gate="G$1" pin="1"/>
+<wire x1="-81.28" y1="-106.68" x2="-83.82" y2="-106.68" width="0.1524" layer="91"/>
+<wire x1="-83.82" y1="-106.68" x2="-83.82" y2="-111.76" width="0.1524" layer="91"/>
 </segment>
 <segment>
@@
 <segment>
 <pinref part="3.3V1" gate="G$1" pin="3.3V"/>
+<pinref part="SJ1" gate="G$1" pin="3"/>
+<wire x1="-81.28" y1="-101.6" x2="-83.82" y2="-101.6" width="0.1524" layer="91"/>
+<wire x1="-83.82" y1="-101.6" x2="-83.82" y2="-96.52" width="0.1524" layer="91"/>
+<wire x1="-83.82" y1="-96.52" x2="-86.36" y2="-96.52" width="0.1524" layer="91"/>
+<pinref part="IC1" gate="SPEC" pin="!RST"/>
 <wire x1="-68.58" y1="-101.6" x2="-71.12" y2="-101.6" width="0.1524" layer="91"/>
-<pinref part="IC1" gate="SPEC" pin="!RST"/>
+<wire x1="-71.12" y1="-101.6" x2="-71.12" y2="-96.52" width="0.1524" layer="91"/>
+<wire x1="-71.12" y1="-96.52" x2="-83.82" y2="-96.52" width="0.1524" layer="91"/>
+<junction x="-83.82" y="-96.52"/>
 </segment>
 <segment>
@@
 </segment>
 </net>
-<net name="N$1" class="0">
+<net name="LED_G" class="0">
 <segment>
 <pinref part="X7" gate="G$1" pin="G-"/>
@@
 </segment>
 </net>
-<net name="N$10" class="0">
+<net name="LED_Y" class="0">
 <segment>
 <pinref part="X7" gate="G$1" pin="Y-"/>
@@
 </segment>
 </net>
-<net name="N$42" class="0">
+<net name="LED_LINK" class="0">
 <segment>
 <wire x1="187.96" y1="-134.62" x2="187.96" y2="-124.46" width="0.1524" layer="91"/>
@@
 </segment>
 </net>
-<net name="N$43" class="0">
+<net name="LED_ACT" class="0">
 <segment>
 <pinref part="R5" gate="G$1" pin="1"/>
@@
 </segment>
 </net>
+<net name="BOOT0" class="0">
+<segment>
+<pinref part="SJ1" gate="G$1" pin="2"/>
+<pinref part="IC1" gate="SPEC" pin="BOOT0"/>
+<wire x1="-76.2" y1="-104.14" x2="-68.58" y2="-104.14" width="0.1524" layer="91"/>
+</segment>
+</net>

Commit message: changed eth socket to HR911105A
Parts:
- X7: device netcat:B78477P1001A014 -> netcat:RJ45-HR11105A
Changed lines of the file:
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@@
 <?xml version="1.0" encoding="utf-8"?>
 <!DOCTYPE eagle SYSTEM "eagle.dtd">
-<eagle version="8.6.3">
+<eagle version="9.0.1">
 <drawing>
 <settings>
@@
 <layer number="59" name="tCarbon" color="7" fill="1" visible="no" active="no"/>
 <layer number="60" name="bCarbon" color="7" fill="1" visible="no" active="no"/>
+<layer number="88" name="SimResults" color="9" fill="1" visible="yes" active="yes"/>
+<layer number="89" name="SimProbes" color="9" fill="1" visible="yes" active="yes"/>
 <layer number="90" name="Modules" color="7" fill="1" visible="no" active="yes"/>
 <layer number="91" name="Nets" color="2" fill="1" visible="yes" active="yes"/>
@@
 <parts>
 <part name="R5" library="netcat" deviceset="RES" device="R0402" value="330"/>
-<part name="X7" library="netcat" deviceset="B78477P" device="1001A014" value="B78477P1001A314"/>
+<part name="X7" library="netcat" deviceset="RJ45" device="-HR11105A" value="B78477P1001A314"/>
 <part name="C3" library="netcat" deviceset="CAP" device="C0402" value="10p"/>
 <part name="R3" library="netcat" deviceset="RES" device="R0402" value="330"/>

Commit message: added solid jumper for RMII/MII clock selecting
Parts:
- added SJ2: (no value), netcat:SJ3
- OSC1: value 25mhz -> 8mhz
- OSC2: value 8mhz -> 25mhz
- TP2: value C -> CLK
Connections:
- removed net N$3: IC2.X1, OSC1.OUT
- new net PHY_OSC: IC2.X1, OSC2.OUT, SJ2.2
- net 3.3V: now also IC1SPEC.VBAT
- net ETH_RX_CLK: now also SJ2.3
- net SYS_CLK: now also OSC1.OUT, SJ2.1; no longer OSC2.OUT
Other:
- moved on the sheet: OSC1, OSC2, SW1
